File: ykb-dactyl-v1.kicad_sch (KiCad schematic)
At the start: 1 part

Commit message: Update
Other:
- added sheet Power (power.kicad_sch)
Changed lines of the file:
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@@
+		)
+	)
+	(sheet
+		(at -304.8 11.43)
+		(size 273.05 220.98)
+		(exclude_from_sim no)
+		(in_bom yes)
+		(on_board yes)
+		(dnp no)
+		(fields_autoplaced yes)
+		(stroke
+			(width 0.1524)
+			(type solid)
+		)
+		(fill
+			(color 0 0 0 0.0000)
+		)
+		(property "Sheetname" "Power"
+			(at -304.8 10.7184 0)
+			(effects
+				(font
+					(size 1.27 1.27)
+				)
+				(justify left bottom)
+			)
+		)
+		(property "Sheetfile" "power.kicad_sch"
+			(at -304.8 232.9946 0)
+			(effects
+				(font
+					(size 1.27 1.27)
+				)
+				(justify left top)
+			)
+		)
+		(instances
+			(project "ykb-dactyl-v1"
+				(path "/e14fa40b-de41-4d68-adfe-82a50bad5819"
+					(page "2")
+				)
+			)
 		)
 	)

Commit message: Update
Parts:
- removed U1: ~, holyiot-21069:holyiot-21069, symbol holyiot-21069:holyiot-21069
Other:
- added sheet Connectors (connectors.kicad_sch)
- added sheet MCU (mcu.kicad_sch)
- added sheet MUXes (muxes.kicad_sch)

Commit message: Update
Other:
- sheet Connectors renamed USB
- sheet USB: file connectors.kicad_sch -> usb.kicad_sch
Changed lines of the file:
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@@
 			(color 0 0 0 0.0000)
 		)
-		(property "Sheetname" "Connectors"
+		(property "Sheetname" "USB"
 			(at 38.1 52.6284 0)
 			(effects
@@
 			)
 		)
-		(property "Sheetfile" "connectors.kicad_sch"
+		(property "Sheetfile" "usb.kicad_sch"
 			(at 38.1 111.0746 0)
 			(effects
