File: mcu.kicad_sch (KiCad schematic)
At the start: 14 parts, among them IC1 TXU0101DCKR, J10 Conn_01x05, J9 Conn_01x05, U1 holyiot-21069

Commit message: Developer Preview 1
Parts:
- U1: now in the parts list

Commit message: Developer Preview 2
Parts:
- removed R4, R5, R6: 10K, Resistor_SMD:R_0402_1005Metric, symbol Device:R_US
- added Q91: BC847BDW1, Package_TO_SOT_SMD:SOT-363_SC-70-6, symbol Transistor_BJT:BC847BDW1
- added Q92: BC847W, Package_TO_SOT_SMD:SOT-323_SC-70, symbol Transistor_BJT:BC847W
- added R91, R93, R95: 100K, Resistor_SMD:R_0402_1005Metric, symbol Device:R_US
- added R92, R94, R96: 47K, Resistor_SMD:R_0402_1005Metric, symbol Device:R_US
- R97: renamed from R1; value 600 -> 10K
- R98: renamed from R2; value 600 -> 10K
- R99: renamed from R3; value 600 -> 5K
Connections:
- net +3.3V_SYS: now also R92.1, R94.1, R96.1; no longer D1.3 (AR), D1.5 (AG), D2.3 (AR), D2.5 (AG)
- net BAT_STAT_1: now also R93.2; no longer U1.P0.17
- net BAT_STAT_1_P: now also U1.P0.17, Q91.6 (C1), R94.2; no longer D1.4 (KR), D2.4 (KR), R97.2
- net BAT_STAT_2: now also R95.2; no longer U1.P0.18
- net BAT_STAT_2_P: now also U1.P0.18, Q91.3 (C2), R96.2; no longer D1.6 (KR), D2.6 (KR), R98.2
- net CHARGER_EN: now also Q92.3 (C), R92.2
- net GND: now also Q91.1 (E1), Q91.4 (E2), Q92.2 (E)
- net ALARMB: no longer names the net of U1.P1.2 (P1.02)
- net DBG_LED_P renamed DBG_LED_LED
- new net: Q91.2 (B1), R93.1
- new net: Q92.1 (B), R91.1
- new net: Q91.5 (B2), R95.1
- new net +5V_USB: R91.2
- new net BAT_STAT_1_LED: D1.4 (KR), D2.4 (KR), R97.2
- new net BAT_STAT_2_LED: D1.6 (KR), D2.6 (KR), R98.2
- new net VCC_PRESYS: D1.3 (AR), D1.5 (AG), D2.3 (AR), D2.5 (AG)
- no-connect marks 17 -> 18
Other:
- moved on the sheet: R97, R98, R99, U1C, U1D, U1E
