File: ykb-skadi-pcb.kicad_pcb (KiCad board)
At the start: 2 copper layers, 55.7 x 57.2 mm, 74 parts, among them IC1 TXU0101DCKR, J1 JST_SH_BM10B-SRSS-TB_1x10-1MP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, J10 Conn_01x05, J11 Conn_01x02_MountingPin, J2 JST_SH_BM10B-SRSS-TB_1x10-1MP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, J3 JST_SH_BM10B-SRSS-TB_1x10-1MP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, J4 JST_SH_BM10B-SRSS-TB_1x10-1MP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, J5 JST_SH_BM10B-SRSS-TB_1x10-1MP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, J6 JST_SH_BM10B-SRSS-TB_1x10-1MP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, J7 JST_SH_BM12B-SRSS-TB_1x12-1MP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

Commit message: Rename the board to Skadi
Other:
- board text added: "SKADI_MB_REV_1.0"
- board text removed: "DV1_MB_REV_1.0"
