File: thumb-board/thumb-board.kicad_sch (KiCad schematic)
At the start: 26 parts, among them IC1 TMAG5253BA1IQDMRR, IC10 TMAG5253BA1IQDMRR, IC11 TMAG5253BA1IQDMRR, IC12 TMAG5253BA1IQDMRR, IC2 TMAG5253BA1IQDMRR, IC3 TMAG5253BA1IQDMRR, IC4 TMAG5253BA1IQDMRR, IC5 TMAG5253BA1IQDMRR, IC6 TMAG5253BA1IQDMRR, IC7 TMAG5253BA1IQDMRR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

Commit message: Developer Preview 1
Parts:
- IC10, IC11, IC12, IC7, IC8, IC9, J2, U10, U11, U12, U7, U8, U9: now not fitted; now left out of the parts list
